Commit message: refactor: Remove not used packages and rename packages for this projects

File: my_robot/urdf/renato_robot.xacro (robot description, xacro)
@@ -1,4 +1,4 @@
 <?xml version='1.0'?>
-<robot name="my_robot"
+<robot name="renato_robot"
   xmlns:xacro="http://www.ros.org/wiki/xacro">
   <!-- #### INERTIA MACROS ####  -->
@@ -13,5 +13,5 @@
   </xacro:macro>
   <link name="robot_footprint"></link>
-  <xacro:include filename="$(find my_robot)/urdf/my_robot.gazebo" />
+  <xacro:include filename="$(find renato_robot)/urdf/renato_robot.gazebo" />
   <joint name="robot_footprint_joint" type="fixed">
     <origin xyz="0 0 0" rpy="0 0 0" />
@@ -223,5 +223,5 @@
     <origin xyz="0 0 0" rpy=" 0 0 0"/>
     <geometry>
-      <mesh filename="package://my_robot/meshes/hokuyo.dae"/>
+      <mesh filename="package://renato_robot/meshes/hokuyo.dae"/>
     </geometry>
   </visual>
